File: Feather_UWB.kicad_pcb (KiCad board)
At the start: 2 copper layers, 50.8 x 22.9 mm, 22 parts, among them J1 Conn_02x03_Counter_Clockwise, J1 feather long, J2 feather short, SW1 RESET

Commit message: Before release
Other:
- board text added: "@Georgia Tech WiSciTech Lab"
